File: ADC.kicad_pcb (KiCad board)
At the start: 2 copper layers, 101.5 x 50.5 mm, 79 parts, among them IC1 ADC0820BCWMX_NOPB, IC2 LCMXO3LF-1300C-5TG100C, IC3 LP38692MPX-3.3_NOPB, IC4 LP38692MPX-5.0_NOPB, J1 Conn_01x06, Y1 ECS-5032MV-320-BN-TR

Commit message: Routed resistors for switch bank. Need to clear DRC
Parts:
- Y1: value ECS-5032MV-320-BN-TR -> ~
- moved R8 5.37 mm to (112.7, 93.3)
- moved R7 5.37 mm to (115.6, 93.3)
- moved R6 5.36 mm to (118.6, 93.3)
- moved R5 5.36 mm to (121.5, 93.3)
- moved R4 5.35 mm to (124.5, 93.3)
- moved R3 5.35 mm to (127.4, 93.3)
- moved R2 5.34 mm to (130.4, 93.3)
- moved R1 5.34 mm to (133.3, 93.3)
Connections:
- R1 pad 1: Net-(R1-Pad1) -> S0
- R2 pad 1: Net-(R2-Pad1) -> S1
- R3 pad 1: Net-(R3-Pad1) -> S2
- R4 pad 1: Net-(R4-Pad1) -> S3
- R5 pad 1: Net-(R5-Pad1) -> S4
- R6 pad 1: Net-(R6-Pad1) -> S5
- R7 pad 1: Net-(R7-Pad1) -> S6
- R8 pad 1: Net-(R8-Pad1) -> S7
- S1 pad 1: Net-(R1-Pad1) -> 3.3V
- S1 pad 2: Net-(R2-Pad1) -> 3.3V
- S1 pad 3: Net-(R3-Pad1) -> 3.3V
- S1 pad 4: Net-(R4-Pad1) -> 3.3V
- S1 pad 5: Net-(R5-Pad1) -> 3.3V
- S1 pad 6: Net-(R6-Pad1) -> 3.3V
- S1 pad 7: Net-(R7-Pad1) -> 3.3V
- S1 pad 8: Net-(R8-Pad1) -> 3.3V
Routing:
- net 3.3V: track 254.8 -> 379.7 mm
- net S1: track 17.8 -> 23.6 mm, vias 0 -> 1
- net S0: track 15.0 -> 20.8 mm, vias 0 -> 1
- net S2: track 20.5 -> 26.0 mm, vias 0 -> 1
- net Net-(R8-Pad1): track 5.32 -> 0.00 mm, vias 1 -> 0
- net S7: track 34.1 -> 39.4 mm, vias 0 -> 1
- net Net-(R1-Pad1): track 5.23 -> 0.00 mm, vias 1 -> 0
- net S3: track 23.2 -> 28.4 mm, vias 0 -> 1
- net Net-(R7-Pad1): track 5.13 -> 0.00 mm, vias 1 -> 0
- net S6: track 31.4 -> 36.5 mm, vias 0 -> 1
- net Net-(R2-Pad1): track 5.04 -> 0.00 mm, vias 1 -> 0
- net S5: track 28.7 -> 33.6 mm, vias 0 -> 1
- net S4: track 25.9 -> 30.9 mm, vias 0 -> 1
- net Net-(R6-Pad1): track 4.94 -> 0.00 mm, vias 1 -> 0
- net Net-(R3-Pad1): track 4.85 -> 0.00 mm, vias 1 -> 0
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Other:
- outline, holes or cut-outs redrawn

Commit message: Completed modifications. Ready for review
Parts:
- removed ? (x3): , 
- removed REF**: MountingHole_2.2mm_M2_DIN965_Pad, MountingHole:MountingHole_2.2mm_M2_DIN965_Pad
- removed TP4: Probe-, TestPoint:TestPoint_THTPad_2.5x2.5mm_Drill1.2mm
Routing:
- net 3.3V: track 379.7 -> 378.8 mm
Other:
- board text removed: "Probe-"

Commit message: Generated fabrication files and moved a few components to pass JLCPCB DFM check
Parts:
- moved C2 6.55 mm to (195.1, 105.5), turned to 90 degrees
Routing:
- net GND: vias 388 -> 386
Other:
- board text added: "Rev 5 - 2026"
- board text added: "Samuel Johnson 2026 Revised by Allen Morrsion"
- board text removed: "Rev 4 - 2026"
- board text removed: "Samuel Johnson 2026"

Commit message: Rewired reset switch to toggle between grounded reset pin and VCC. Corrected some symbol errors
Parts:
- turned S2 to 180 degrees
Connections:
- R9 pad 1: Net-(S2-COM_1) -> RST
- S2 pad 1: Net-(S2-COM_1) -> 3.3V
Routing:
- net 3.3V: track 378.8 -> 392.5 mm
- net Net-(S2-COM_1): track 11.0 -> 0.00 mm, vias 1 -> 0
- net RST: track 19.6 -> 19.3 mm, vias 0 -> 1
